Commit message: restructuring

File: urdf/ur5e.urdf (robot description, URDF)
Before this commit: robot ur5e, 11 links, 10 joints
Links:
- link base_link: geometry collision mesh filename=file://$(find ur5_pick_and_place)/meshes/collision/base.stl scale=1.0 1.0 1.0; visual mesh filename=file://$(find ur5_pick_and_place)/meshes/visual/base.dae
- link forearm_link: geometry collision mesh filename=file://$(find ur5_pick_and_place)/meshes/collision/forearm.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 scale=1.0 1.0 1.0; visual mesh filename=file://$(find ur5_pick_and_place)/meshes/visual/forearm.dae
- link shoulder_link: geometry collision mesh filename=file://$(find ur5_pick_and_place)/meshes/collision/shoulder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 scale=1.0 1.0 1.0; visual mesh filename=file://$(find ur5_pick_and_place)/meshes/visual/shoulder.dae
- link upper_arm_link: geometry collision mesh filename=file://$(find ur5_pick_and_place)/meshes/collision/upperarm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 scale=1.0 1.0 1.0; visual mesh filename=file://$(find ur5_pick_and_place)/meshes/visual/upperarm.dae
- link wrist_1_link: geometry collision mesh filename=file://$(find ur5_pick_and_place)/meshes/collision/wrist1.s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 scale=1.0 1.0 1.0; visual mesh filename=file://$(find ur5_pick_and_place)/meshes/visual/wrist1.dae
- link wrist_2_link: geometry collision mesh filename=file://$(find ur5_pick_and_place)/meshes/collision/wrist2.s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 scale=1.0 1.0 1.0; visual mesh filename=file://$(find ur5_pick_and_place)/meshes/visual/wrist2.dae
- link wrist_3_link: geometry collision mesh filename=file://$(find ur5_pick_and_place)/meshes/collision/wrist3.s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 scale=1.0 1.0 1.0; visual mesh filename=file://$(find ur5_pick_and_place)/meshes/visual/wrist3.dae
